Commit message: fix: macos adaptation

File: description/robot_description/urdf/robot_description.urdf.xacro (robot description, xacro)
@@ -309,5 +309,5 @@
     <child link="lower_arm"/>
     <axis xyz="0 0 1"/>
-    <limit effort="10" velocity="10" lower="-1.74533" upper="1.5708"/>
+    <limit effort="10" velocity="10" lower="-1.178" upper="1.178"/>
   </joint>
   <joint name="Wrist_Pitch" type="revolute">

File: description/ros2_control/so_arm101_ros2_control.xacro (robot description, xacro)
@@ -19,10 +19,10 @@
         <param name="bus_id">1</param>
         <param name="servo_type">300</param>
-        <param name="offset_deg">0</param>
+        <param name="offset_deg">200</param>
         <param name="direction">1</param>
         <param name="scale">1</param>
         <param name="servo_min_deg">80</param>
         <param name="servo_max_deg">320</param>
-        <param name="servo_default_deg">0</param>
+        <param name="servo_default_deg">200</param>
         <command_interface name="position">
           <param name="min">-1.91986</param>
@@ -36,10 +36,10 @@
         <param name="bus_id">2</param>
         <param name="servo_type">300</param>
-        <param name="offset_deg">0</param>
+        <param name="offset_deg">182.5</param>
         <param name="direction">1</param>
         <param name="scale">1</param>
         <param name="servo_min_deg">75</param>
         <param name="servo_max_deg">290</param>
-        <param name="servo_default_deg">0</param>
+        <param name="servo_default_deg">182.5</param>
         <command_interface name="position">
           <param name="min">-1.74533</param>
@@ -53,13 +53,13 @@
         <param name="bus_id">3</param>
         <param name="servo_type">300</param>
-        <param name="offset_deg">0</param>
+        <param name="offset_deg">207.5</param>
         <param name="direction">1</param>
         <param name="scale">1</param>
         <param name="servo_min_deg">140</param>
         <param name="servo_max_deg">275</param>
-        <param name="servo_default_deg">0</param>
+        <param name="servo_default_deg">207.5</param>
         <command_interface name="position">
-          <param name="min">-1.74533</param>
-          <param name="max">1.5708</param>
+          <param name="min">-1.178</param>
+          <param name="max">1.178</param>
         </command_interface>
         <state_interface name="position" />
@@ -70,10 +70,10 @@
         <param name="bus_id">4</param>
         <param name="servo_type">300</param>
-        <param name="offset_deg">0</param>
+        <param name="offset_deg">177.5</param>
         <param name="direction">1</param>
         <param name="scale">1</param>
         <param name="servo_min_deg">74</param>
         <param name="servo_max_deg">281</param>
-        <param name="servo_default_deg">0</param>
+        <param name="servo_default_deg">177.5</param>
         <command_interface name="position">
           <param name="min">-1.65806</param>
@@ -87,10 +87,10 @@
         <param name="bus_id">5</param>
         <param name="servo_type">300</param>
-        <param name="offset_deg">0</param>
+        <param name="offset_deg">90</param>
         <param name="direction">1</param>
         <param name="scale">1</param>
         <param name="servo_min_deg">0</param>
         <param name="servo_max_deg">360</param>
-        <param name="servo_default_deg">0</param>
+        <param name="servo_default_deg">180</param>
         <command_interface name="position">
           <param name="min">-2.79253</param>
@@ -104,10 +104,10 @@
         <param name="bus_id">6</param>
         <param name="servo_type">300</param>
-        <param name="offset_deg">0</param>
+        <param name="offset_deg">137.5</param>
         <param name="direction">1</param>
         <param name="scale">1</param>
         <param name="servo_min_deg">115</param>
         <param name="servo_max_deg">250</param>
-        <param name="servo_default_deg">0</param>
+        <param name="servo_default_deg">137.5</param>
         <command_interface name="position">
           <param name="min">-0.174533</param>

Commit message: evol(limit): widen the Elbow to its measured travel
The elbow could not fold far enough because the URDF stopped it at +-1.178 rad,
well inside the joint's real range. That figure was never measured: the servo
window that shipped with it, 140-275 deg about an offset of 207.5, restates
+-67.5 deg exactly, so the window was derived from the URDF rather than the
hardware and the two agreed only because one was copied from the other.

The follower calibration recorded 866-3083 ticks about a 2048 centre, which is
-103.89 .. +90.97 deg -- about 195 deg of travel against the 135 the URDF
allowed. Use those hard stops, so the URDF and the servo clamp now bound the
joint at the same place.

File: description/robot_description/urdf/robot_description.urdf.xacro (robot description, xacro)
@@ -309,5 +309,8 @@
     <child link="lower_arm"/>
     <axis xyz="0 0 1"/>
-    <limit effort="10" velocity="10" lower="-1.178" upper="1.178"/>
+    <!-- Hard stops recorded by the follower calibration (866..3083 ticks about a
+         2048 centre). The previous +-1.178 was a guess: the servo window shipped
+         alongside it restated the same number, so nothing here was measured. -->
+    <limit effort="10" velocity="10" lower="-1.81317" upper="1.58767"/>
   </joint>
   <joint name="Wrist_Pitch" type="revolute">

File: description/ros2_control/so_arm101_ros2_control.xacro (robot description, xacro)
@@ -60,6 +60,6 @@
         <param name="servo_default_deg">180</param>
         <command_interface name="position">
-          <param name="min">-1.178</param>
-          <param name="max">1.178</param>
+          <param name="min">-1.81317</param>
+          <param name="max">1.58767</param>
         </command_interface>
         <state_interface name="position" />

Commit message: Hardware support (#2)
* evol(limit): update limit

Signed-off-by: m-brl <103381146+m-brl@users.noreply.github.com>

* fix(so_arm101): own the spawners, leave the controller_manager to the supervisor

control.launch.py started its own ros2_control_node as well as including
lucy_control_supervisor, which owns one. The supervisor saw a controller_manager
it did not start and refused to bring the stack up rather than drive the same
joints twice. Drop the local one; inmoov already delegates it.

Chain the spawners on process exit instead of staggering them by index*2
seconds. A spawner holds a global lock while waiting for controller_manager, so
overlapping ones each burn a full 20s lock attempt; chaining also removes the
guess at how long the supervisor takes to answer. use_sim_time went with the
fixed delays: this file only runs off Gazebo.

control.launch.yaml named an entry xacro that does not exist
(so_arm101.urdf.xacro); the file is robot.urdf.xacro. Bringup resolves urdf_path
through this file, so the wrong name is what pushed lucy.launch.py into
hardcoding a path.

* fix(so_arm101): shorten hardware node_name and set it in both modes

macOS caps POSIX shared-memory and semaphore names at 30 bytes, and the hardware
interface derives three names from node_name. lucy_hardware_interface_so_arm
made "/lucy_hardware_interface_so_arm.lucy_reg_table" 46 bytes, so shm_open
failed with ENAMETOOLONG and the component never initialised.

The param also sat inside xacro:unless use_mock_hardware, so it vanished in mock
mode and the hardware fell back to its built-in default. Set it on <hardware>
where it applies to both.

Note this file is generated by lucy_config_generator and marked do-not-edit, so
regenerating drops this; the generator does not emit bus_servo or bus_id either,
which is why the checked-in copy already diverges from config/hardware/active.yaml.

* fix: limits of ros2_control xacro

* fix: macos adaptation

* evol(calibration): take servo windows from the LeRobot follower calibration

The servo_*_deg fields are degrees on the scale the firmware maps onto raw
STS3215 ticks: BusServoConfig in firmwares/rp2040 spans 0-360 deg over
0-4096 pulse, so deg = ticks * 360/4096. Mathieu's windows were already in
that space (wrist_roll 0-360 against a recorded 0-4095 confirms the scale),
they were just measured on a different arm.

Convert the recorded ranges and set offset_deg to 180. The calibration writes
a homing offset that centres each joint on 2048 ticks, so 180 deg is the homed
pose rather than the window midpoint the previous values assumed: every URDF
joint span now falls inside its servo window, and the jaw lands at 179.82 for
fully closed against a URDF zero of 0 rad.

direction stays 1 everywhere. The five arm windows are symmetric about 2048 and
say nothing about which way the joint turns; only the jaw is pinned, its window
sitting above centre because it opens. Flip the joints that run backwards
against the 3D view once the arm is on the bench.

* evol(limit): widen the Elbow to its measured travel

The elbow could not fold far enough because the URDF stopped it at +-1.178 rad,
well inside the joint's real range. That figure was never measured: the servo
window that shipped with it, 140-275 deg about an offset of 207.5, restates
+-67.5 deg exactly, so the window was derived from the URDF rather than the
hardware and the two agreed only because one was copied from the other.

The follower calibration recorded 866-3083 ticks about a 2048 centre, which is
-103.89 .. +90.97 deg -- about 195 deg of travel against the 135 the URDF
allowed. Use those hard stops, so the URDF and the servo clamp now bound the
joint at the same place.

* fix(lint): satisfy pep257 and flake8 in control.launch.py

Same D213 as inmoov_urdf on the spawner docstring, plus E303/E305 from the
blank lines around controllers_to_spawn. ament_lint_common runs both linters
here too, so this branch would have failed CI the moment it was pushed.

* feat(scripts): apply a LeRobot calibration to the hardware config

lerobot-calibrate records each servo's travel in raw STS3215 ticks; the hardware
YAML wants the same windows in degrees on the scale the firmware maps onto ticks
(BusServoConfig spans 0-360 deg over 0-4096 pulse). Converting six joints by
hand invites a transposed digit that only shows up as a joint driving into its
stop, so do it in code.

Records pair with actuators by servo bus id against physical_pin. The keys in
the file are LeRobot's own joint names and say nothing about urdf_joint, so a
name match would be a guess; a record that pairs with nothing aborts the run
before anything is written, since a half-applied calibration drives some joints
against a window measured for others.

offset_deg becomes 180 deg, the 2048-tick centre the calibration homes each
joint to, rather than the midpoint of the window -- those coincide only where
travel happens to be symmetric, which the gripper's is not. direction is left
alone: it is verified against the 3D view on hardware, and drive_mode describes
an inversion relative to LeRobot's URDF rather than ours, so a non-zero value is
reported instead of applied.

Edits are textual, so comments and key order survive. Generated artefacts are
left to the generator.

Tests cover the tick scale, id matching, comment survival, idempotence, and the
rejection paths, and round-trip the committed config: the recorded ticks
reproduce config/hardware/active.yaml byte for byte.

* fix: point the stale references at robot.urdf.xacro

The entry xacro was renamed from so_arm101.urdf.xacro in 262a944, but nine
references to the old name stayed behind. test_xacro_smoke asserted on a path
that no longer exists, so both of its cases failed outright wherever xacro is on
PATH -- CI included. joint_preview.launch.py and gazebo.launch.py pointed at the
same missing file, and the developer guide documented it in four places.

* chore: trimmed comment

* refactor(scripts): stop patching the xacro from the calibration script

The generator can emit the bus_servo params now, so the ros2_control xacro
is generated again and patching it here only duplicated what regeneration
does. It also never touched gazebo.xacro, which is why Gazebo kept running
on the previous calibration. Regenerating afterwards is now required, and
the docs say so.

Drops the incidental bug where --config pointed at another file still
rewrote the package's own xacro.

* chore(hardware): move so_arm to bus_servo_only and recalibrate

Also carries a fresh LeRobot calibration for the arm now on the bench, so
the servo windows differ from the previous one throughout.

The ros2_control xacro is regenerated rather than hand-edited: its params
come out identical to the hand-maintained file, except each joint keeps the
virtual_pin slot active.yaml already assigned it instead of all six being
flattened to 0.

* chore: removed pycache

* docs: install the generated firmware layout when regenerating

* fix(ci): add github actions build-and-test workflow (#3)

* fix(lint): wrap long usage line for flake8 E501

* fix(ci): add gitHub actions build-and-test workflow

* fix(ci): call org robot-package reusable workflow

* chore: trimmed comments

* chore: removed pycache

* chore: ament_copyright and ament_flake8

* chore: ament_copyright

* chore: white space

---------

Signed-off-by: m-brl <103381146+m-brl@users.noreply.github.com>
Co-authored-by: m-brl <103381146+m-brl@users.noreply.github.com>
Co-authored-by: Charles Madjeri <80175305+charlesmadjeri@users.noreply.github.com>

File: description/robot_description/urdf/robot_description.urdf.xacro (robot description, xacro)
@@ -309,5 +309,5 @@
     <child link="lower_arm"/>
     <axis xyz="0 0 1"/>
-    <limit effort="10" velocity="10" lower="-1.74533" upper="1.5708"/>
+    <limit effort="10" velocity="10" lower="-1.81317" upper="1.58767"/>
   </joint>
   <joint name="Wrist_Pitch" type="revolute">

File: description/ros2_control/so_arm101_ros2_control.xacro (robot description, xacro)
@@ -11,16 +11,18 @@
       <xacro:unless value="$(arg use_mock_hardware)">
         <param name="publisher_topic">actuators/so_arm</param>
-        <param name="node_name">lucy_hardware_interface_so_arm</param>
+        <param name="node_name">so_arm</param>
       </xacro:unless>
     </hardware>
       <joint name="Rotation">
+          <param name="type">bus_servo</param>
           <param name="virtual_pin">0</param>
+          <param name="bus_id">1</param>
           <param name="servo_type">300</param>
-          <param name="offset_deg">0</param>
+          <param name="offset_deg">180</param>
           <param name="direction">1</param>
           <param name="scale">1</param>
-          <param name="servo_min_deg">-110</param>
-          <param name="servo_max_deg">110</param>
-          <param name="servo_default_deg">0</param>
+          <param name="servo_min_deg">62.31</param>
+          <param name="servo_max_deg">283.8</param>
+          <param name="servo_default_deg">180</param>
           <command_interface name="position">
             <param name="min">-1.91986</param>
@@ -30,12 +32,14 @@
       </joint>
       <joint name="Pitch">
+          <param name="type">bus_servo</param>
           <param name="virtual_pin">1</param>
+          <param name="bus_id">2</param>
           <param name="servo_type">300</param>
-          <param name="offset_deg">0</param>
+          <param name="offset_deg">180</param>
           <param name="direction">1</param>
           <param name="scale">1</param>
-          <param name="servo_min_deg">-100</param>
-          <param name="servo_max_deg">100</param>
-          <param name="servo_default_deg">0</param>
+          <param name="servo_min_deg">73.65</param>
+          <param name="servo_max_deg">282.13</param>
+          <param name="servo_default_deg">180</param>
           <command_interface name="position">
             <param name="min">-1.74533</param>
@@ -45,27 +49,31 @@
       </joint>
       <joint name="Elbow">
+          <param name="type">bus_servo</param>
           <param name="virtual_pin">2</param>
+          <param name="bus_id">3</param>
           <param name="servo_type">300</param>
-          <param name="offset_deg">0</param>
+          <param name="offset_deg">180</param>
           <param name="direction">1</param>
           <param name="scale">1</param>
-          <param name="servo_min_deg">-100</param>
-          <param name="servo_max_deg">90</param>
-          <param name="servo_default_deg">0</param>
+          <param name="servo_min_deg">74.27</param>
+          <param name="servo_max_deg">271.14</param>
+          <param name="servo_default_deg">180</param>
           <command_interface name="position">
-            <param name="min">-1.74533</param>
-            <param name="max">1.5708</param>
+            <param name="min">-1.81317</param>
+            <param name="max">1.58767</param>
           </command_interface>
           <state_interface name="position" />
       </joint>
       <joint name="Wrist_Pitch">
+          <param name="type">bus_servo</param>
           <param name="virtual_pin">3</param>
+          <param name="bus_id">4</param>
           <param name="servo_type">300</param>
-          <param name="offset_deg">0</param>
+          <param name="offset_deg">180</param>
           <param name="direction">1</param>
           <param name="scale">1</param>
-          <param name="servo_min_deg">-95</param>
-          <param name="servo_max_deg">95</param>
-          <param name="servo_default_deg">0</param>
+          <param name="servo_min_deg">70.14</param>
+          <param name="servo_max_deg">279.76</param>
+          <param name="servo_default_deg">180</param>
           <command_interface name="position">
             <param name="min">-1.65806</param>
@@ -75,12 +83,14 @@
       </joint>
       <joint name="Wrist_Roll">
+          <param name="type">bus_servo</param>
           <param name="virtual_pin">4</param>
+          <param name="bus_id">5</param>
           <param name="servo_type">300</param>
-          <param name="offset_deg">0</param>
+          <param name="offset_deg">180</param>
           <param name="direction">1</param>
           <param name="scale">1</param>
-          <param name="servo_min_deg">-160</param>
-          <param name="servo_max_deg">160</param>
-          <param name="servo_default_deg">0</param>
+          <param name="servo_min_deg">0</param>
+          <param name="servo_max_deg">359.91</param>
+          <param name="servo_default_deg">180</param>
           <command_interface name="position">
             <param name="min">-2.79253</param>
@@ -90,12 +100,14 @@
       </joint>
       <joint name="Jaw">
+          <param name="type">bus_servo</param>
           <param name="virtual_pin">5</param>
+          <param name="bus_id">6</param>
           <param name="servo_type">300</param>
-          <param name="offset_deg">0</param>
+          <param name="offset_deg">180</param>
           <param name="direction">1</param>
           <param name="scale">1</param>
-          <param name="servo_min_deg">-10</param>
-          <param name="servo_max_deg">100</param>
-          <param name="servo_default_deg">0</param>
+          <param name="servo_min_deg">178.68</param>
+          <param name="servo_max_deg">309.81</param>
+          <param name="servo_default_deg">180</param>
           <command_interface name="position">
             <param name="min">-0.174533</param>
